File: openpwm.kicad_pcb (KiCad board)
At the start: 2 copper layers, 148.8 x 42.7 mm, 134 parts, among them J1 Conn_01x04, J10 Conn_01x04, J11 Conn_01x04, J12 Conn_01x04, J13 Conn_01x04, J14 Conn_01x04, J15 Conn_01x04, J16 Conn_01x04, J17 PSU MOLEX 1, J18 PSU MOLEX 2, J19 USB HEADER, J2 Conn_01x04, J20 Cortex Debug Connector, J21 TSENSE_1, J22 TSENSE_2, J23 TSENSE_3, J24 TSENSE_4, J3 Conn_01x04, J4 Conn_01x04, J5 Conn_01x04, J6 Conn_01x04, J7 Conn_01x04, J8 Conn_01x04, J9 Conn_01x04, U1 TPS62111, U2 TM4C123GE6PM, U3 LSF0108, U4 LSF0108, U5 TLP291-4, U6 TLP291-4, U7 TLP291-4, U8 TLP291-4, Y1 Crystal

Commit message: Start the PCB layout
This commit starts the PCB layout. There is still a long way to go;
just using this as checkpoint.
Parts:
- J19: footprint Pin_Headers:Pin_Header_Straight_1x04_Pitch2.00mm -> Pin_Headers:Pin_Header_Straight_1x04_Pitch2.54mm
- Y1: footprint Crystals:Crystal_SMD_HC49-SD_HandSoldering -> Crystals:Crystal_SMD_5032-2pin_5.0x3.2mm_HandSoldering
- moved R55 108.3 mm to (56.0, 50.8)
- moved R77 107.9 mm to (88.6, 36.1)
- moved R67 107.9 mm to (52.2, 62.2)
- moved R79 105.1 mm to (101.4, 36.6), turned to 180 degrees
- moved R60 104.4 mm to (56.0, 58.2)
- moved C5 101.7 mm to (90.7, 49.3), turned to 180 degrees
- moved R78 101.0 mm to (95.3, 36.1), turned to 180 degrees
- moved C1 98.7 mm to (164.8, 64.5), turned to 90 degrees
- moved C2 98.2 mm to (99.8, 38.1), turned to 180 degrees
- moved C15 95.6 mm to (113.5, 43.4), turned to 90 degrees
- moved R80 93.3 mm to (106.4, 37.5), turned to 90 degrees
- moved C8 92.5 mm to (99.1, 56.1), turned to 180 degrees
- moved R45 91.8 mm to (92.5, 60.6), turned to 270 degrees
- moved C20 90.2 mm to (111.1, 45.2)
- moved C9 88.2 mm to (99.1, 59.2), turned to 180 degrees
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- renumbered 1uF1 to C20
Connections:
- net /USB_D+ renamed USB_D+
- net /USB_D- renamed USB_D-
- R61 pad 1: +12V -> +12VA
- R62 pad 1: +12V -> +12VA
- R63 pad 1: +12V -> +12VA
- R64 pad 1: +12V -> +12VA
- R65 pad 1: +12V -> +12VA
- R66 pad 1: +12V -> +12VA
- R67 pad 1: +12V -> +12VA
- R68 pad 1: +12V -> +12VA
- U2 pad 32: Net-(U2-Pad32) -> GND
- U2 pad 6: /TSENSE_4 -> /TSENSE_3
- U2 pad 63: /TSENSE_1 -> /TSENSE_2
- U2 pad 64: /TSENSE_2 -> /TSENSE_1
- U2 pad 9: /TSENSE_3 -> /TSENSE_4
Routing:
- net GND: track 0.00 -> 75.0 mm, vias 0 -> 48
- net /TSENSE_4: track 0.00 -> 49.8 mm
- net +5V: track 0.00 -> 44.9 mm
- net /TSENSE_3: track 0.00 -> 41.0 mm
- net USB_D-: track 0.00 -> 14.9 mm
- net /TSENSE_1: track 0.00 -> 14.5 mm
- net USB_D+: track 0.00 -> 11.7 mm
- net Net-(C14-Pad1): track 0.00 -> 10.6 mm
- net /TSENSE_2: track 0.00 -> 10.2 mm
- net /V_DDC: track 0.00 -> 9.94 mm
- net /PWM3_C4: track 0.00 -> 9.69 mm
- net +5VA: track 0.00 -> 8.20 mm
- net /USB0VBUS: track 0.00 -> 7.98 mm
- net /PWM3_C3: track 0.00 -> 7.89 mm
- net Net-(L1-Pad1): track 0.00 -> 7.57 mm
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- added copper zone on F.Cu, net +12V
- added copper zone on F.Cu, net +12VA
- added copper zone on F.Cu, net +3V3
Other:
- net class Default: clearance 0.2 -> 0.1524; trace_width 0.25 -> 0.1524; via_dia 0.6 -> 0.6858; via_drill 0.4 -> 0.3302
- rule pad_to_mask_clearance: 0.2 -> 0.0508
- rule trace_clearance: 0.2 -> 0.1524
- rule trace_min: 0.2 -> 0.1524
- rule via_min_drill: 0.3 -> 0.3302
- rule via_min_size: 0.4 -> 0.6858

Commit message: 70 nets to go
Parts:
- moved R65 127.0 mm to (48.0, 57.8), turned to 270 degrees
- moved R62 125.4 mm to (43.4, 57.8), turned to 270 degrees
- moved R61 125.0 mm to (41.9, 57.8), turned to 270 degrees
- moved R56 123.1 mm to (56.0, 45.7)
- moved R58 122.2 mm to (56.0, 41.1)
- moved R52 121.2 mm to (56.1, 33.5), turned to 270 degrees
- moved R57 120.7 mm to (56.0, 36.6)
- moved R64 118.3 mm to (46.5, 57.8), turned to 270 degrees
- moved R54 118.2 mm to (56.0, 39.6)
- moved R53 117.9 mm to (56.0, 38.1)
- moved R59 117.3 mm to (56.0, 44.2)
- moved R63 116.4 mm to (45.0, 57.8), turned to 270 degrees
- moved R68 113.2 mm to (52.6, 57.8), turned to 270 degrees
- moved R66 112.7 mm to (49.5, 57.8), turned to 270 degrees
- moved R70 103.2 mm to (84.2, 42.2), turned to 180 degrees
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Connections:
- U1 pad 17: (no net) -> GND
Routing:
- net /PWM_A1: track 0.00 -> 60.5 mm, vias 0 -> 2
- net /PWM_A4: track 0.00 -> 60.3 mm, vias 0 -> 2
- net /PWM_A3: track 0.00 -> 59.4 mm, vias 0 -> 2
- net /PWM_A2: track 0.00 -> 56.9 mm, vias 0 -> 2
- net Net-(R52-Pad1): track 0.00 -> 52.7 mm
- net Net-(R35-Pad1): track 0.00 -> 52.6 mm
- net /JTAG_TDO: track 0.00 -> 46.2 mm
- net Net-(R61-Pad2): track 0.00 -> 41.7 mm
- net Net-(R62-Pad2): track 0.00 -> 37.4 mm
- net Net-(R5-Pad2): track 0.00 -> 37.1 mm
- net Net-(R63-Pad2): track 0.00 -> 33.1 mm
- net Net-(R4-Pad2): track 0.00 -> 32.7 mm
- net /RPM_D1: track 0.00 -> 29.8 mm
- net /RPM_A1: track 0.00 -> 29.7 mm
- net /RPM_B1: track 0.00 -> 29.1 mm
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
Commit message: Fix optocoupler schematic
Connections:
- net /USB0ID renamed Net-(U2-Pad45)
- net USB_D+ renamed /USBD_P
- net USB_D- renamed /USBD_N
- U1 pad 17: GND -> (no net)
- U5 pad 10: +3V3 -> /RPM3_A4
- U5 pad 12: +3V3 -> /RPM3_A3
- U5 pad 14: +3V3 -> /RPM3_A2
- U5 pad 16: +3V3 -> /RPM3_A1
- U6 pad 10: +3V3 -> /RPM3_B4
- U6 pad 12: +3V3 -> /RPM3_B3
- U6 pad 14: +3V3 -> /RPM3_B2
- U6 pad 16: +3V3 -> /RPM3_B1
- U7 pad 10: +3V3 -> /RPM3_C4
- U7 pad 12: +3V3 -> /RPM3_C3
- U7 pad 14: +3V3 -> /RPM3_C2
- U7 pad 16: +3V3 -> /RPM3_C1
- U8 pad 10: +3V3 -> /RPM3_D4
- U8 pad 12: +3V3 -> /RPM3_D3
- U8 pad 14: +3V3 -> /RPM3_D2
- U8 pad 16: +3V3 -> /RPM3_D1
Routing:
- net GND: vias 55 -> 51
- net (no net): vias 0 -> 4
